Commit message: attemt to fix tf

File: src/go2_description/urdf/go2.urdf (robot description, URDF)
Before this commit: robot go2_description, 31 links, 30 joints
Links:
- added link base_link
Joints:
- added joint base_link_joint: type fixed, parent base_link, child base, origin xyz=0 0 0 rpy=0 0 0, axis 0 0 0
- joint camera_link_joint: parent base -> base_link
- joint imu_joint: parent base -> base_link
- joint lidar_frame_joint: origin xyz=0.0018320158435115 0.000108320625906232 0.253633251213134 rpy=0 0 0 -> xyz=0.28945 0 -0.046825 rpy=0 2.8782 0; parent base -> base_link
- joint radar_joint: origin xyz=0.28945 0 -0.046825 rpy=0 2.8782 0 -> xyz=0 0 0 rpy=0 0 0; parent base -> lidar_frame
